Commit message: Modify for use with DJI Matrice

File: hector_quadrotor_description/urdf/quadrotor_base.urdf.xacro (robot description, xacro)
@@ -1,6 +1,7 @@
 <?xml version="1.0"?>
 <robot xmlns:xacro="http://www.ros.org/wiki/xacro">
-  <xacro:include filename="$(find hector_sensors_description)/urdf/sonar_sensor.urdf.xacro" />
+  <!-- <xacro:include filename="$(find hector_sensors_description)/urdf/sonar_sensor.urdf.xacro" /> -->
   <xacro:property name="pi" value="3.1415926535897931" />
+  <xacro:include filename="$(find dji_m100_description)/urdf/dji_m100_base.xacro" />
   <!-- Main quadrotor link -->
   <xacro:macro name="quadrotor_base_macro">
@@ -14,5 +15,6 @@
         <origin xyz="0 0 0" rpy="0 0 0" />
         <geometry>
-          <mesh filename="package://hector_quadrotor_description/meshes/quadrotor/quadrotor_base.dae"/>
+          <!-- <mesh filename="package://hector_quadrotor_description/meshes/quadrotor/quadrotor_base.dae"/> -->
+	  <mesh filename="package://dji_m100_description/meshes/dji_m100/dji_m100.dae"/>
         </geometry>
       </visual>
@@ -20,12 +22,13 @@
         <origin xyz="0 0 0" rpy="0 0 0" />
         <geometry>
-          <mesh filename="package://hector_quadrotor_description/meshes/quadrotor/quadrotor_base.stl"/>
+          <!-- <mesh filename="package://hector_quadrotor_description/meshes/quadrotor/quadrotor_base.stl"/> -->
+	  <mesh filename="package://dji_m100_description/meshes/dji_m100/dji_m100.stl"/>
         </geometry>
       </collision>
     </link>
     <!-- Sonar height sensor -->
-    <xacro:sonar_sensor name="sonar" parent="base_link" ros_topic="sonar_height" update_rate="10" min_range="0.03" max_range="3.0" field_of_view="${40*pi/180}" ray_count="3">
+    <!-- <xacro:sonar_sensor name="sonar" parent="base_link" ros_topic="sonar_height" update_rate="10" min_range="0.03" max_range="3.0" field_of_view="${40*pi/180}" ray_count="3">
       <origin xyz="-0.16 0.0 -0.012" rpy="0 ${90*pi/180} 0"/>
-    </xacro:sonar_sensor>
+    </xacro:sonar_sensor> -->
   </xacro:macro>
 </robot>

File: hector_quadrotor_gazebo/urdf/quadrotor_sensors.gazebo.xacro (robot description, xacro)
@@ -39,6 +39,6 @@
             <bodyName>base_link</bodyName>
             <frameId>$(arg base_link_frame)</frameId>
-            <topicName>fix</topicName>
-            <velocityTopicName>fix_velocity</velocityTopicName>
+            <topicName>gps</topicName>
+            <velocityTopicName>gps_velocity</velocityTopicName>
             <referenceLatitude>49.860246</referenceLatitude>
             <referenceLongitude>8.687077</referenceLongitude>
